File: antenna_analyser.sch (KiCad schematic (older format))
At the start: 27 parts, among them IC1 MCP6002, IC2 ARDUINO_PRO_MINI_3.3V, P1 AD9850_CONN, P2 BNC, P3 CONN_LCD, U1 AMS1117

Commit message: Added a USB micro connector, and a 14-pin strip socket for the LCD.
Parts:
- removed P3: CONN_LCD, symbol CONN_01X09
- removed PWR1: CONN_01X02, Wire_Connections_Bridges:WireConnection_1mmDrill, symbol CONN_01X02
- added P3: CONN_LCD, Socket_Strips:Socket_Strip_Straight_1x14, symbol CONN_01X14
- added P4: USB_OTG, Connect:USB_Micro-B, symbol USB_OTG
Connections:
- wire segments 130 -> 129
Changed lines of the file:
@@
 $EndDescr
 $Comp
-L +5V #PWR8
+L +5V #PWR01
 U 1 1 5570837F
 P 5450 6250
-F 0 "#PWR8" H 5450 6100 50  0001 C CNN
+F 0 "#PWR01" H 5450 6100 50  0001 C CNN
 F 1 "+5V" H 5450 6390 50  0000 C CNN
 F 2 "" H 5450 6250 60  0000 C CNN
@@
 $EndComp
 $Comp
-L GND #PWR6
+L GND #PWR02
 U 1 1 5570893A
 P 4900 6250
-F 0 "#PWR6" H 4900 6000 50  0001 C CNN
+F 0 "#PWR02" H 4900 6000 50  0001 C CNN
 F 1 "GND" H 4900 6100 50  0000 C CNN
 F 2 "" H 4900 6250 60  0000 C CNN
@@
 $EndComp
 $Comp
-L GND #PWR5
+L GND #PWR03
 U 1 1 55708C34
 P 4050 6250
-F 0 "#PWR5" H 4050 6000 50  0001 C CNN
+F 0 "#PWR03" H 4050 6000 50  0001 C CNN
 F 1 "GND" H 4050 6100 50  0000 C CNN
 F 2 "" H 4050 6250 60  0000 C CNN
@@
 $EndComp
 $Comp
-L GND #PWR9
+L GND #PWR04
 U 1 1 55717CB8
 P 5650 1950
-F 0 "#PWR9" H 5650 1700 50  0001 C CNN
+F 0 "#PWR04" H 5650 1700 50  0001 C CNN
 F 1 "GND" H 5650 1800 50  0000 C CNN
 F 2 "" H 5650 1950 60  0000 C CNN
@@
 $EndComp
 $Comp
-L GND #PWR10
+L GND #PWR05
 U 1 1 55718CAB
 P 5650 6250
-F 0 "#PWR10" H 5650 6000 50  0001 C CNN
+F 0 "#PWR05" H 5650 6000 50  0001 C CNN
 F 1 "GND" H 5650 6100 50  0000 C CNN
 F 2 "" H 5650 6250 60  0000 C CNN
@@
 $EndComp
 $Comp
-L GND #PWR13
+L GND #PWR06
 U 1 1 558DD57F
 P 7950 2000
-F 0 "#PWR13" H 7950 1750 50  0001 C CNN
+F 0 "#PWR06" H 7950 1750 50  0001 C CNN
 F 1 "GND" H 7950 1850 50  0000 C CNN
 F 2 "" H 7950 2000 60  0000 C CNN
@@
 	8950 2750 8950 1350
 Wire Wire Line
-	8750 1350 10150 1350
+	10150 1350 8750 1350
 Wire Wire Line
 	7950 1850 7950 2000
 $Comp
-L +5V #PWR12
+L +5V #PWR07
 U 1 1 558DD6BD
 P 7000 700
-F 0 "#PWR12" H 7000 550 50  0001 C CNN
+F 0 "#PWR07" H 7000 550 50  0001 C CNN
 F 1 "+5V" H 7000 840 50  0000 C CNN
 F 2 "" H 7000 700 60  0000 C CNN
@@
 	7000 700  7000 1350
 $Comp
-L GND #PWR11
+L GND #PWR08
 U 1 1 558DDC04
 P 6450 2050
-F 0 "#PWR11" H 6450 1800 50  0001 C CNN
+F 0 "#PWR08" H 6450 1800 50  0001 C CNN
 F 1 "GND" H 6450 1900 50  0000 C CNN
 F 2 "" H 6450 2050 60  0000 C CNN
@@
 $EndComp
 $Comp
-L +5V #PWR1
+L +5V #PWR09
 U 1 1 558F3FBC
 P 1200 3450
-F 0 "#PWR1" H 1200 3300 50  0001 C CNN
+F 0 "#PWR09" H 1200 3300 50  0001 C CNN
 F 1 "+5V" H 1200 3590 50  0000 C CNN
 F 2 "" H 1200 3450 60  0000 C CNN
@@
 $EndComp
 $Comp
-L GND #PWR2
+L GND #PWR010
 U 1 1 558F41B6
 P 1200 4800
-F 0 "#PWR2" H 1200 4550 50  0001 C CNN
+F 0 "#PWR010" H 1200 4550 50  0001 C CNN
 F 1 "GND" H 1200 4650 50  0000 C CNN
 F 2 "" H 1200 4800 60  0000 C CNN
@@
 Connection ~ 5250 4800
 $Comp
-L GND #PWR7
+L GND #PWR011
 U 1 1 558F649D
 P 5250 6250
-F 0 "#PWR7" H 5250 6000 50  0001 C CNN
+F 0 "#PWR011" H 5250 6000 50  0001 C CNN
 F 1 "GND" H 5250 6100 50  0000 C CNN
 F 2 "" H 5250 6250 60  0000 C CNN
@@
 Connection ~ 7000 850
 $Comp
-L GND #PWR16
+L GND #PWR012
 U 1 1 55904F2C
 P 9550 2050
-F 0 "#PWR16" H 9550 1800 50  0001 C CNN
+F 0 "#PWR012" H 9550 1800 50  0001 C CNN
 F 1 "GND" H 9550 1900 50  0000 C CNN
 F 2 "" H 9550 2050 60  0000 C CNN
@@
 $EndComp
 Wire Wire Line
-	9550 2050 9550 1200
-Wire Wire Line
-	9650 1200 9650 2100
+	9550 1050 9550 2050
+Wire Wire Line
+	9650 1050 9650 2100
 Wire Wire Line
 	9650 2100 9750 2100
@@
 	9750 2100 9750 2750
 Wire Wire Line
-	9950 1200 9950 2200
+	9950 1050 9950 2200
 Wire Wire Line
 	9950 2200 9650 2200
@@
 	9650 2200 9650 2750
 Wire Wire Line
-	10050 1200 10050 2300
+	10050 1050 10050 2300
 Wire Wire Line
 	10050 2300 9450 2300
@@
 	9450 2300 9450 2750
 Wire Wire Line
-	10150 1350 10150 1200
+	10150 1050 10150 1350
 Connection ~ 8950 1350
 Wire Wire Line
-	10250 1200 10250 2400
+	10250 1050 10250 2400
 Wire Wire Line
 	10250 2400 9550 2400
@@
 	9350 6200 9350 4400
 $Comp
-L GND #PWR15
+L GND #PWR013
 U 1 1 5597D150
 P 8950 5750
-F 0 "#PWR15" H 8950 5500 50  0001 C CNN
+F 0 "#PWR013" H 8950 5500 50  0001 C CNN
 F 1 "GND" H 8950 5600 50  0000 C CNN
 F 2 "" H 8950 5750 60  0000 C CNN
@@
 $EndComp
 $Comp
-L CONN_01X02 PWR1
-U 1 1 559C0ACF
-P 2550 900
-F 0 "PWR1" H 2550 1050 50  0000 C CNN
-F 1 "CONN_01X02" V 2650 900 50  0000 C CNN
-F 2 "Wire_Connections_Bridges:WireConnection_1mmDrill" H 2550 900 60  0001 C CNN
-F 3 "" H 2550 900 60  0000 C CNN
-	1    2550 900
-	1    0    0    -1
-$EndComp
-$Comp
-L +5V #PWR3
+L +5V #PWR014
 U 1 1 559C0C97
-P 2200 750
-F 0 "#PWR3" H 2200 600 50  0001 C CNN
-F 1 "+5V" H 2200 890 50  0000 C CNN
-F 2 "" H 2200 750 60  0000 C CNN
-F 3 "" H 2200 750 60  0000 C CNN
-	1    2200 750
-	1    0    0    -1
-$EndComp
-$Comp
-L GND #PWR4
+P 1650 2750
+F 0 "#PWR014" H 1650 2600 50  0001 C CNN
+F 1 "+5V" H 1650 2890 50  0000 C CNN
+F 2 "" H 1650 2750 60  0000 C CNN
+F 3 "" H 1650 2750 60  0000 C CNN
+	1    1650 2750
+	-1   0    0    1
+$EndComp
+$Comp
+L GND #PWR015
 U 1 1 559C0CCB
-P 2200 1050
-F 0 "#PWR4" H 2200 800 50  0001 C CNN
-F 1 "GND" H 2200 900 50  0000 C CNN
-F 2 "" H 2200 1050 60  0000 C CNN
-F 3 "" H 2200 1050 60  0000 C CNN
-	1    2200 1050
-	1    0    0    -1
-$EndComp
-Wire Wire Line
-	2350 950  2200 950
-Wire Wire Line
-	2200 950  2200 1050
-Wire Wire Line
-	2200 750  2200 850
-Wire Wire Line
-	2200 850  2350 850
+P 2050 2750
+F 0 "#PWR015" H 2050 2500 50  0001 C CNN
+F 1 "GND" H 2050 2600 50  0000 C CNN
+F 2 "" H 2050 2750 60  0000 C CNN
+F 3 "" H 2050 2750 60  0000 C CNN
+	1    2050 2750
+	1    0    0    -1
+$EndComp
 $Comp
 L BNC P2
@@
 	5100 1400 6300 1400
 Wire Wire Line
-	9750 1200 9750 1900
+	9750 1050 9750 1900
 Wire Wire Line
 	9750 1900 9150 1900
@@
 	9150 1900 9150 2750
 Wire Wire Line
-	9850 1200 9850 1800
+	9850 1050 9850 1800
 Wire Wire Line
 	9850 1800 9050 1800
@@
 	9050 1800 9050 2750
 $Comp
-L GND #PWR14
+L GND #PWR016
 U 1 1 55A1262A
 P 8950 5300
-F 0 "#PWR14" H 8950 5050 50  0001 C CNN
+F 0 "#PWR016" H 8950 5050 50  0001 C CNN
 F 1 "GND" H 8950 5150 50  0000 C CNN
 F 2 "" H 8950 5300 60  0000 C CNN
@@
 	8950 5550 8950 5750
 $Comp
-L GND #PWR17
+L GND #PWR017
 U 1 1 55A12973
 P 11000 5750
-F 0 "#PWR17" H 11000 5500 50  0001 C CNN
+F 0 "#PWR017" H 11000 5500 50  0001 C CNN
 F 1 "GND" H 11000 5600 50  0000 C CNN
 F 2 "" H 11000 5750 60  0000 C CNN
@@
 	1200 4200 1200 4800
 $Comp
-L CONN_01X09 P3
-U 1 1 55A1397C
-P 9850 1000
-F 0 "P3" H 9850 1500 50  0000 C CNN
-F 1 "CONN_LCD" V 9950 1000 50  0000 C CNN
-F 2 "" H 9850 1000 60  0000 C CNN
-F 3 "" H 9850 1000 60  0000 C CNN
-	1    9850 1000
+L USB_OTG P4
+U 1 1 55C68FD7
+P 1850 2150
+F 0 "P4" H 2175 2025 50  0000 C CNN
+F 1 "USB_OTG" H 1850 2350 50  0000 C CNN
+F 2 "Connect:USB_Micro-B" V 1800 2050 60  0001 C CNN
+F 3 "" V 1800 2050 60  0000 C CNN
+	1    1850 2150
+	1    0    0    -1
+$EndComp
+Wire Wire Line
+	1650 2750 1650 2450
+Wire Wire Line
+	2050 2450 2050 2750
+$Comp
+L CONN_01X14 P3
+U 1 1 55C698D3
+P 10100 850
+F 0 "P3" H 10100 1600 50  0000 C CNN
+F 1 "CONN_LCD" V 10200 850 50  0000 C CNN
+F 2 "Socket_Strips:Socket_Strip_Straight_1x14" H 10100 850 60  0001 C CNN
+F 3 "" H 10100 850 60  0000 C CNN
+	1    10100 850
 	0    -1   -1   0
 $EndComp
+Wire Wire Line
+	9450 1200 9450 1050
 $EndSCHEMATC

Commit message: Added programming connector.
Parts:
- added P5: CONN_PROG, Socket_Strips:Socket_Strip_Straight_1x04, symbol CONN_01X04
Connections:
- net GND: now also P5.4 (P4)
- net at IC2.1 (TX0): now also P5.1 (P1)
- net at IC2.2 (RX1): now also P5.2 (P2)
- net at IC2.3 (RST): now also P5.3 (P3)
Changed lines of the file:
@@
 Wire Wire Line
 	9450 1200 9450 1050
+$Comp
+L CONN_01X04 P5
+U 1 1 55C6A4DD
+P 8100 4200
+F 0 "P5" H 8100 4450 50  0000 C CNN
+F 1 "CONN_PROG" V 8200 4200 50  0000 C CNN
+F 2 "Socket_Strips:Socket_Strip_Straight_1x04" H 8100 4200 60  0001 C CNN
+F 3 "" H 8100 4200 60  0000 C CNN
+	1    8100 4200
+	0    -1   -1   0
+$EndComp
+Wire Wire Line
+	8250 4400 8250 4500
+Wire Wire Line
+	8250 4500 8950 4500
+Connection ~ 8950 4500
+Wire Wire Line
+	8150 4400 8150 4600
+Wire Wire Line
+	8150 4600 8850 4600
+Wire Wire Line
+	8850 4600 8850 4400
+Wire Wire Line
+	8050 4400 8050 4700
+Wire Wire Line
+	8050 4700 8750 4700
+Wire Wire Line
+	8750 4700 8750 4400
+Wire Wire Line
+	8650 4400 8650 4800
+Wire Wire Line
+	8650 4800 7950 4800
+Wire Wire Line
+	7950 4800 7950 4400
 $EndSCHEMATC
