File: antenna_analyser.kicad_pcb (KiCad board)
At the start: 2 copper layers, 100 x 50 mm, 32 parts, among them IC1 MCP6002, IC2 ARDUINO_PRO_MINI_3.3V, P1 AD9850_CONN, P2 BNC, P3 CONN_LCD, P4 USB_OTG, P5 CONN_PROG, U1 AMS1117

Commit message: Added auxiliary soldering points to make it easier to attach the USB socket to the board.
Parts:
- added ?: , Measurement_Points:Measurement_Point_Square-SMD-Pad_Big, B.Cu at (102.2, 130.0)
- added ?: S, Measurement_Points:Measurement_Point_Square-SMD-Pad_Big, B.Cu at (111.0, 130.0)
Changed lines of the file:
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@@
     (tracks 306)
     (zones 0)
-    (modules 32)
+    (modules 34)
     (nets 54)
   )
@@
     (mod_text_size 1 1)
     (mod_text_width 0.15)
-    (pad_size 1.35 0.4)
+    (pad_size 2.99974 2.99974)
     (pad_drill 0)
     (pad_to_mask_clearance 0)
@@
     (add_net "Net-(C5-Pad1)")
   )
+  (module Measurement_Points:Measurement_Point_Square-SMD-Pad_Big (layer B.Cu)
+    (at 102.25 130)
+    (descr "Mesurement Point, Square, SMD Pad,  3mm x 3mm,")
+    (tags "Mesurement Point, Square, SMD Pad, 3mm x 3mm,")
+    (fp_text reference "" (at 0 3.81) (layer B.SilkS)
+      (effects (font (size 1 1) (thickness 0.15)) (justify mirror))
+    )
+    (fp_text value "" (at 2.54 -3.81) (layer B.Fab)
+      (effects (font (size 1 1) (thickness 0.15)) (justify mirror))
+    )
+    (pad Sold smd rect (at 0 0) (size 2.99974 2.99974) (layers B.Cu B.Paste B.Mask))
+  )
   (module dds-module-ad9850:DDS_AD9850 locked (layer F.Cu)
     (at 136.6 108.9 270)
@@
     )
   )
+  (module Measurement_Points:Measurement_Point_Square-SMD-Pad_Big (layer B.Cu)
+    (at 111 130)
+    (descr "Mesurement Point, Square, SMD Pad,  3mm x 3mm,")
+    (tags "Mesurement Point, Square, SMD Pad, 3mm x 3mm,")
+    (fp_text reference "" (at 0 3.81) (layer B.SilkS)
+      (effects (font (size 1 1) (thickness 0.15)) (justify mirror))
+    )
+    (fp_text value S (at 2.54 -3.81) (layer B.Fab) hide
+      (effects (font (size 1 1) (thickness 0.15)) (justify mirror))
+    )
+    (pad Sold smd rect (at 0 0) (size 2.99974 2.99974) (layers B.Cu B.Paste B.Mask))
+  )
   (gr_text http://j.mp/HFAA9850 (at 113.35 87.1) (layer F.Cu)

Commit message: Production artifacts.
Routing:
- added copper zone on B.Cu, net GND
- added copper zone on F.Cu, net GND
Changed lines of the file:
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@@
-(kicad_pcb (version 4) (host pcbnew "(2015-06-03 BZR 5697)-product")
+(kicad_pcb (version 4) (host pcbnew 4.0.6)
   (general
     (links 72)
     (no_connects 0)
-    (area 70.714287 64.15 223 159.700001)
+    (area 70.864287 64.3 222.85 159.700001)
     (thickness 1.6)
     (drawings 9)
@@
     (pad_to_mask_clearance 0)
     (aux_axis_origin 0 0)
-    (visible_elements FFFFFF7F)
+    (visible_elements FFFFEF7F)
     (pcbplotparams
-      (layerselection 0x00000_80000000)
+      (layerselection 0x3ffff_80000001)
       (usegerberextensions false)
       (excludeedgelayer true)
@@
       (padsonsilk false)
       (subtractmaskfromsilk false)
-      (outputformat 4)
+      (outputformat 1)
       (mirror false)
-      (drillshape 2)
+      (drillshape 0)
       (scaleselection 1)
-      (outputdirectory production/))
+      (outputdirectory gerber))
   )
   (net 0 "")
@@
   (segment (start 109.3201 128.1314) (end 110.1009 128.9122) (width 0.4) (layer F.Cu) (net 53))
   (segment (start 109.1009 128.1314) (end 109.3201 128.1314) (width 0.4) (layer F.Cu) (net 53))
+  (zone (net 5) (net_name GND) (layer F.Cu) (hatch edge 0.508)
+    (connect_pads (clearance 0.508))
+    (min_thickness 0.254)
+    (fill yes (arc_segments 16) (thermal_gap 0.508) (thermal_bridge_width 0.508))
+    (polygon
+      (pts
+        (xy 90 84) (xy 190 84) (xy 190 134) (xy 90 134)
+      )
+    )
+  )
+  (zone (net 5) (net_name GND) (layer B.Cu) (hatch edge 0.508)
+    (connect_pads (clearance 0.508))
+    (min_thickness 0.254)
+    (fill yes (arc_segments 16) (thermal_gap 0.508) (thermal_bridge_width 0.508))
+    (polygon
+      (pts
+        (xy 90 84) (xy 190 84) (xy 190 134) (xy 90 134)
+      )
+    )
+  )
 )
